File: hardware/ib4/ib4.kicad_pcb (KiCad board)
At the start: 4 copper layers, 23 parts, among them J1 Conn_01x02_Female, J2 Screw_Terminal_01x02, J3 Screw_Terminal_01x02, J6 Screw_Terminal_01x03, J7 Screw_Terminal_01x03, J9 Screw_Terminal_01x03, Q1 Q_NPN_EBC, Q2 Q_PNP_BCE, U1 DC-DC_5V_TSR_1-22450, U2 tpl5110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

Commit message: update
Parts:
- removed H3: MountingHole, MountingHole:MountingHole_2.7mm_M2.5
- moved H4 141.9 mm to (20.0, 68.0)
- moved H2 34.6 mm to (102.0, 68.0)
- moved J7 31.6 mm to (31.9, 66.8), turned to 0 degrees
- moved H1 30.8 mm to (102.0, -2.00)
- moved J6 21.4 mm to (25.6, 9.00)
- moved U6 18.4 mm to (21.3, -1.60)
- moved R3 7.64 mm to (42.2, 42.4)
- moved J1 6.08 mm to (28.4, 45.9)
- moved U2 5.80 mm to (33.7, 40.9)
Routing:
- net GND: track 229.5 -> 190.8 mm
- net 5V_BUCK: track 49.9 -> 80.9 mm
- net D9: track 88.0 -> 112.1 mm, vias 0 -> 2
- net TIMER: track 60.2 -> 40.2 mm
- net +3V3: track 299.1 -> 282.9 mm, vias 4 -> 6
- net DONE: track 35.6 -> 37.3 mm
- net Net-(J1-Pad1): track 5.87 -> 5.28 mm
Other:
- board outline added: 95.3 x 82.3 mm
